File: ece411_t2_schematic.sch (EAGLE design)
At the start: 0 parts

Commit message: Add files via upload
Parts:
- added J1: AVR_SPI_PROG_3X2PTH, SparkFun-Connectors:AVR_SPI_PROG_3X2PTH
- added T1, T2, T3, T4: 2N3904, transistor:2N3904
- added U1: 328P, SparkFun-IC-Microcontroller:ATMEGA328P_PDIP
Connections:
- new net GND: J1.6, U1.GND
- new net MISO: J1.1, U1.PB4(MISO)
- new net MOSI: J1.4, U1.PB3(MOSI/OC2)
- new net N$3: T1.B, U1.PB0(ICP)
- new net N$4: T1.E, T2.B
- new net N$5: T3.B, U1.PB1(OC1A)
- new net N$6: T3.E, T4.B
- new net RST: J1.5, U1.PC6(/RESET)
- new net SCK: J1.3, U1.PB5(SCK)
- new net VCC: J1.2, T1.C, T2.C, T3.C, T4.C, U1.AREF, U1.AVCC, U1.VCC
