File: ece411_t2_schematic.sch (EAGLE design)
At the start: 6 parts, among them J1 AVR_SPI_PROG_3X2PTH, T1 2N3904, T2 2N3904, T3 2N3904, T4 2N3904, U1 328P

Commit message: Add files via upload
Parts:
- added C1: 0.1uF, SparkFun-Capacitors:0.1UF-0402-6.3V-10%-X7R
- added J2, J3: (no value), SparkFun-Retired:CONN_02
- added J5, J6, J7: 455-1750-1-ND, SparkFun-Connectors:CONN_03
- added R1: 10k, SparkFun-Resistors:10KOHM-0402-1/16W-1%
- added SV1: (no value), con-lstb:MA04-1
Connections:
- new net N$1: T1.B, U1.PD6(AIN0)
- new net N$10: J5.2
- new net N$11: J7.2
- new net N$12: J6.2
- new net N$13: SV1.1
- new net N$2: T3.B, U1.PD7(AIN1)
- new net N$7: J5.1, U1.PD2(INT0)
- new net N$8: J7.1, U1.PD1(TXD)
- new net N$9: J6.1, U1.PD0(RXD)
- net GND: now also J2.2, J3.2, J5.3, J6.3, J7.3, SV1.4
- net N$3: now also J2.1, T4.E; no longer T1.B, U1.PB0(ICP)
- net N$5: now also J3.1, T2.E; no longer T3.B, U1.PB1(OC1A)
Other:
- moved on the sheet: J1, T1, T2, T3, T4, U1
